File: _autosave-Waterbox 2.1-backups/_autosave-Waterbox 2.1-2024-01-06_181332/Waterbox 2.1.kicad_sch (KiCad schematic)
At the start: 23 parts, among them J1 Jack-DC

Commit message: route tracks in back copper, adding dc jack for additional dc power connector
Parts:
- added 5V1: TP1, TestPoint:TestPoint_Pad_D1.5mm, symbol Connector:TestPoint
- added GND1: TP2, TestPoint:TestPoint_Pad_D1.5mm, symbol Connector:TestPoint
- H1, H2, H3: footprint MountingHole:MountingHole_3.5mm -> MountingHole:MountingHole_3mm
- H4, H5, H6, H7, H8: footprint MountingHole:MountingHole_3.5mm_Pad_Via -> MountingHole:MountingHole_3mm_Pad_Via
Connections:
- net +5V: now also 5V1.1
- net GND: now also GND1.1
Changed lines of the file:
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@@
   (junction (at 218.44 39.37) (diameter 0) (color 0 0 0 0)
   )
+  (junction (at 125.73 24.13) (diameter 0) (color 0 0 0 0)
+  )
   (junction (at 41.91 24.13) (diameter 0) (color 0 0 0 0)
   )
   (junction (at 257.81 15.24) (diameter 0) (color 0 0 0 0)
   )
+  (junction (at 125.73 31.75) (diameter 0) (color 0 0 0 0)
+  )
   (junction (at 257.81 20.32) (diameter 0) (color 0 0 0 0)
   )
@@
     (stroke (width 0) (type default))
   )
+  (wire (pts (xy 128.27 24.13) (xy 125.73 24.13))
+    (stroke (width 0) (type default))
+  )
   (wire (pts (xy 257.81 25.4) (xy 271.78 25.4))
     (stroke (width 0) (type default))
@@
     (stroke (width 0) (type default))
   )
+  (wire (pts (xy 118.11 31.75) (xy 125.73 31.75))
+    (stroke (width 0) (type default))
+  )
   (wire (pts (xy 36.83 99.06) (xy 36.83 101.6))
     (stroke (width 0) (type default))
@@
     (stroke (width 0) (type default))
   )
-  (wire (pts (xy 118.11 24.13) (xy 128.27 24.13))
+  (wire (pts (xy 118.11 24.13) (xy 125.73 24.13))
     (stroke (width 0) (type default))
   )
@@
     (stroke (width 0) (type default))
   )
+  (wire (pts (xy 125.73 20.32) (xy 125.73 24.13))
+    (stroke (width 0) (type default))
+  )
   (wire (pts (xy 209.55 54.61) (xy 222.25 54.61))
     (stroke (width 0) (type default))
   )
-  (wire (pts (xy 118.11 31.75) (xy 128.27 31.75))
+  (wire (pts (xy 128.27 31.75) (xy 125.73 31.75))
     (stroke (width 0) (type default))
   )
@@
   )
   (wire (pts (xy 44.45 99.06) (xy 36.83 99.06))
+    (stroke (width 0) (type default))
+  )
+  (wire (pts (xy 125.73 31.75) (xy 125.73 35.56))
     (stroke (width 0) (type default))
   )
@@
     )
   )
+  (symbol (lib_id "Connector:TestPoint") (at 125.73 20.32 0) (unit 1)
+    (in_bom yes) (on_board yes) (dnp no) (fields_autoplaced)
+    (property "Reference" "5V1" (at 128.27 15.748 0)
+      (effects (font (size 1.27 1.27)) (justify left))
+    )
+    (property "Value" "TP1" (at 128.27 18.288 0)
+      (effects (font (size 1.27 1.27)) (justify left))
+    )
+    (property "Footprint" "TestPoint:TestPoint_Pad_D1.5mm" (at 130.81 20.32 0)
+      (effects (font (size 1.27 1.27)) hide)
+    )
+    (property "Datasheet" "~" (at 130.81 20.32 0)
+      (effects (font (size 1.27 1.27)) hide)
+    )
+    (pin "1")
+    (instances
+      (project "Waterbox 2.1"
+        (path "/779bb994-918f-485e-a5a1-689218580d86"
+          (reference "5V1") (unit 1)
+        )
+      )
+    )
+  )
   (symbol (lib_id "Mechanical:MountingHole_Pad") (at 274.32 20.32 270) (mirror x) (unit 1)
     (in_bom yes) (on_board yes) (dnp no)
@@
       (effects (font (size 1.27 1.27)) hide)
     )
-    (property "Footprint" "MountingHole:MountingHole_3.5mm" (at 274.32 20.32 0)
+    (property "Footprint" "MountingHole:MountingHole_3mm" (at 274.32 20.32 0)
       (effects (font (size 1.27 1.27)) hide)
     )
@@
       (effects (font (size 1.27 1.27)) hide)
     )
-    (property "Footprint" "MountingHole:MountingHole_3.5mm_Pad_Via" (at 274.32 30.48 0)
+    (property "Footprint" "MountingHole:MountingHole_3mm_Pad_Via" (at 274.32 30.48 0)
       (effects (font (size 1.27 1.27)) hide)
     )
@@
       (effects (font (size 1.27 1.27)) hide)
     )
-    (property "Footprint" "MountingHole:MountingHole_3.5mm_Pad_Via" (at 241.3 20.32 0)
+    (property "Footprint" "MountingHole:MountingHole_3mm_Pad_Via" (at 241.3 20.32 0)
       (effects (font (size 1.27 1.27)) hide)
     )
@@
       (effects (font (size 1.27 1.27)) hide)
     )
-    (property "Footprint" "MountingHole:MountingHole_3.5mm" (at 274.32 25.4 0)
+    (property "Footprint" "MountingHole:MountingHole_3mm" (at 274.32 25.4 0)
       (effects (font (size 1.27 1.27)) hide)
     )
@@
       (effects (font (size 1.27 1.27)) hide)
     )
-    (property "Footprint" "MountingHole:MountingHole_3.5mm_Pad_Via" (at 241.3 30.48 0)
+    (property "Footprint" "MountingHole:MountingHole_3mm_Pad_Via" (at 241.3 30.48 0)
       (effects (font (size 1.27 1.27)) hide)
     )
@@
       (effects (font (size 1.27 1.27)) hide)
     )
-    (property "Footprint" "MountingHole:MountingHole_3.5mm" (at 274.32 15.24 0)
+    (property "Footprint" "MountingHole:MountingHole_3mm" (at 274.32 15.24 0)
       (effects (font (size 1.27 1.27)) hide)
     )
@@
       (effects (font (size 1.27 1.27)) hide)
     )
-    (property "Footprint" "MountingHole:MountingHole_3.5mm_Pad_Via" (at 241.3 25.4 0)
+    (property "Footprint" "MountingHole:MountingHole_3mm_Pad_Via" (at 241.3 25.4 0)
       (effects (font (size 1.27 1.27)) hide)
     )
@@
       (effects (font (size 1.27 1.27)) hide)
     )
-    (property "Footprint" "MountingHole:MountingHole_3.5mm_Pad_Via" (at 241.3 15.24 0)
+    (property "Footprint" "MountingHole:MountingHole_3mm_Pad_Via" (at 241.3 15.24 0)
       (effects (font (size 1.27 1.27)) hide)
     )
@@
         )
       )
+    )
+  )
+  (symbol (lib_id "Connector:TestPoint") (at 125.73 35.56 0) (mirror x) (unit 1)
+    (in_bom yes) (on_board yes) (dnp no)
+    (property "Reference" "GND1" (at 128.27 40.132 0)
+      (effects (font (size 1.27 1.27)) (justify left))
+    )
+    (property "Value" "TP2" (at 128.27 37.592 0)
+      (effects (font (size 1.27 1.27)) (justify left))
+    )
+    (property "Footprint" "TestPoint:TestPoint_Pad_D1.5mm" (at 130.81 35.56 0)
+      (effects (font (size 1.27 1.27)) hide)
+    )
+    (property "Datasheet" "~" (at 130.81 35.56 0)
+      (effects (font (size 1.27 1.27)) hide)
+    )
+    (pin "1")
+    (instances
+      (project "Waterbox 2.1"
+        (path "/779bb994-918f-485e-a5a1-689218580d86"
+          (reference "GND1") (unit 1)
+        )
+      )
